Commit message: Add map frame for robots.

File: lft_simulation/urdf/simulation_leader_waking_robot.xacro (robot description, xacro)
@@ -12,4 +12,10 @@
         </inertial>
     </xacro:macro>
+    <link name="${type}_base_footprint" />
+    <joint name="${type}_base_joint" type="fixed">
+        <parent link="${type}_base_footprint" />
+        <child link="${type}_base_link" />
+        <origin xyz="0.0 0.0 0.0919" rpy="0 0 0" />
+    </joint>
     <link name="${type}_base_link">
         <visual>
@@ -183,5 +189,7 @@
             <publish_rate>100</publish_rate>
             <publish_odom>true</publish_odom>
-            <publish_odom_tf>false</publish_odom_tf>
+            <publish_odom_tf>true</publish_odom_tf>
+            <odometry_frame>/${type}/odom</odometry_frame>
+            <robot_base_frame>${type}_base_footprint</robot_base_frame>
             <leftFrontJoint>${type}_base_to_wheel1</leftFrontJoint>
             <rightFrontJoint>${type}_base_to_wheel3</rightFrontJoint>

File: lft_simulation/urdf/simulation_slave_waking_robot.xacro (robot description, xacro)
@@ -12,4 +12,10 @@
         </inertial>
     </xacro:macro>
+    <link name="${type}_base_footprint" />
+    <joint name="${type}_base_joint" type="fixed">
+        <parent link="${type}_base_footprint" />
+        <child link="${type}_base_link" />
+        <origin xyz="0.0 0.0 0.0919" rpy="0 0 0" />
+    </joint>
     <link name="${type}_base_link">
         <visual>
@@ -183,5 +189,7 @@
             <publish_rate>100</publish_rate>
             <publish_odom>true</publish_odom>
-            <publish_odom_tf>false</publish_odom_tf>
+            <publish_odom_tf>true</publish_odom_tf>
+            <odometry_frame>/${type}/odom</odometry_frame>
+            <robot_base_frame>${type}_base_footprint</robot_base_frame>
             <leftFrontJoint>${type}_base_to_wheel1</leftFrontJoint>
             <rightFrontJoint>${type}_base_to_wheel3</rightFrontJoint>

Commit message: 齐次控制未转换坐标系

File: lft_simulation/urdf/simulation_leader_waking_robot.xacro (robot description, xacro)
@@ -8,6 +8,6 @@
         <inertial>
             <mass value="${mass}" />
-            <inertia ixx="0.01" ixy="0.0" ixz="0.0"
-                    iyy="0.01" iyz="0.0" izz="0.01" />
+            <inertia ixx="0.1" ixy="0.0" ixz="0.0"
+                    iyy="0.1" iyz="0.0" izz="0.1" />
         </inertial>
     </xacro:macro>
